File: FTDI_Debug.kicad_sch (KiCad schematic)
At the start: 30 parts, among them J4 10 Pin Cortex Program & Debug, J5 PN, SW2 218-8LPST, U16 AT93C46DN-SH-T, U5 FT4232HQ-Tray, Y1 H130B-12.000-16-2525-EXT-TR

Commit message: Title block improvements
Improved the info in the title blocks, compacted the root sheet to fit on the same size paper as everything else
Other:
- company: (none) -> NewAE Technology
- title: <Enter Sheet Title> -> NAE-SONATA-ONE
Changed lines of the file:
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@@
 	(paper "A3")
 	(title_block
-		(title "<Enter Sheet Title>")
+		(title "NAE-SONATA-ONE")
+		(date "2024-08-16")
+		(rev "10")
+		(company "NewAE Technology")
+		(comment 2 "Apache-2")
 	)
 	(junction
