File: Header_Pins.kicad_sch (KiCad schematic)
At the start: 19 parts, among them J1 SM04B-SRSS-TB_LF__SN_, J7 SM04B-SRSS-TB_LF__SN_, P1 Header 8, P11 Header 3X2, P12 Header 4X2, P2 Header 8, P3 Header 20X2, P4 Header 10, P5 Header 6, P6 Header 8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

Commit message: Title block improvements
Improved the info in the title blocks, compacted the root sheet to fit on the same size paper as everything else
Other:
- company: (none) -> NewAE Technology
- title: <Enter Sheet Title> -> NAE-SONATA-ONE
Changed lines of the file:
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@@
 	(paper "A3")
 	(title_block
-		(title "<Enter Sheet Title>")
+		(title "NAE-SONATA-ONE")
+		(date "2024-08-16")
+		(rev "10")
+		(company "NewAE Technology")
+		(comment 2 "Apache-2")
 	)
 	(junction
