File: LEDs_Switches.kicad_sch (KiCad schematic)
At the start: 57 parts, among them Q3 BSS138, SW4 1-1825058-9, SW5 EVP-ASDC1A, SW7 CUS-13TB, SW8 2425755-1

Commit message: Title block improvements
Improved the info in the title blocks, compacted the root sheet to fit on the same size paper as everything else
Other:
- company: (none) -> NewAE Technology
- title: <Enter Sheet Title> -> NAE-SONATA-ONE
Changed lines of the file:
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@@
 	(paper "A3")
 	(title_block
-		(title "<Enter Sheet Title>")
+		(title "NAE-SONATA-ONE")
+		(date "2024-08-16")
+		(rev "10")
+		(company "NewAE Technology")
+		(comment 2 "Apache-2")
 	)
 	(junction
