File: Main_USB.kicad_sch (KiCad schematic)
At the start: 17 parts, among them J2 USB4105-GF-A, Q1 DMP2123LQ-7, Q4 DMP2123LQ-7, Q5 DMP2123LQ-7, U1 PRTR5V0U2AX

Commit message: Title block improvements
Improved the info in the title blocks, compacted the root sheet to fit on the same size paper as everything else
Other:
- company: (none) -> NewAE Technology
- title: <Enter Sheet Title> -> NAE-SONATA-ONE
Changed lines of the file:
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@@
 	(paper "A3")
 	(title_block
-		(title "<Enter Sheet Title>")
+		(title "NAE-SONATA-ONE")
+		(date "2024-08-16")
+		(rev "10")
+		(company "NewAE Technology")
+		(comment 2 "Apache-2")
 	)
 	(junction
