File: RS485_232_ETH.kicad_sch (KiCad schematic)
At the start: 25 parts, among them J3 J00-0045NL, U3 ISL83485IBZ-T, U7 MAX3221IPWR

Commit message: Title block improvements
Improved the info in the title blocks, compacted the root sheet to fit on the same size paper as everything else
Other:
- company: (none) -> NewAE Technology
- title: <Enter Sheet Title> -> NAE-SONATA-ONE
Changed lines of the file:
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@@
 	(paper "A3")
 	(title_block
-		(title "<Enter Sheet Title>")
+		(title "NAE-SONATA-ONE")
+		(date "2024-08-16")
+		(rev "10")
+		(company "NewAE Technology")
+		(comment 2 "Apache-2")
 	)
 	(junction
